File: Electrical/CAD/Primary/Primary.sch (KiCad schematic (older format))
At the start: 15 parts, among them Q1 2N3904, Q2 2N3906, SW1 SW_DPST, U1 LMC555xN, U2 MCP6282

Commit message: Update the PCB using the bezier curve spiral coil component. See primary-pcb-coil-bezier.png for a preview of the result.
It requires using the latest Nightly Development Builds from https://kicad-downloads.s3.cern.ch/index.html?prefix=windows/nightly/.
However, as noted in the previous commit, it will be very very slow to load (>15 minutes).
I have a patch for this issue that I will submit.
In the meantime, if anyone is interested to use this please contact me and I will send it to you.
Parts:
- BT1: symbol WirelessPower:2x_Battery_Cell -> Primary-rescue:2x_Battery_Cell-WirelessPower
- L1: footprint Jumper:SolderJumper-2_P1.3mm_Open_Pad1.0x1.5mm -> WirelessPower:CoilSpiral_25_Bezier
